Commit message: fix: stabilize osracer lab training tasks

File: source/osracer_lab_assets/data/Robots/OSRacer/osracer.urdf (robot description, URDF)
Before this commit: robot osracer, 11 links, 10 joints
Links:
- link Left_front_wheel_link: geometry collision mesh filename=meshes/Left_front_wheel_link.STL; visual mesh filename=meshes/Left_front_wheel_link.STL
- link base_link: geometry collision mesh filename=meshes/base_link.STL; visual mesh filename=meshes/base_link.STL
- link camera_link: geometry collision mesh filename=meshes/camera_link.STL; visual mesh filename=meshes/camera_link.STL
- link imu_link: geometry collision mesh filename=meshes/imu_link.STL; visual mesh filename=meshes/imu_link.STL
- link laser: geometry collision mesh filename=meshes/laser_link.STL; visual mesh filename=meshes/laser_link.STL
- link left_rear_wheel_link: geometry collision mesh filename=meshes/left_rear_wheel_link.STL; visual mesh filename=meshes/left_rear_wheel_link.STL
- link left_steering_hinge_link: geometry collision mesh filename=meshes/left_steering_hinge_link.STL; visual mesh filename=meshes/left_steering_hinge_link.STL
- link right_front_wheel_link: geometry collision mesh filename=meshes/right_front_wheel_link.STL; visual mesh filename=meshes/right_front_wheel_link.STL
- link right_rear_wheel_link: geometry collision mesh filename=meshes/right_rear_wheel_link.STL; visual mesh filename=meshes/right_rear_wheel_link.STL
- link right_steering_hinge_link: geometry collision mesh filename=meshes/right_steering_hinge_link.STL; visual mesh filename=meshes/right_steering_hinge_link.STL
